File: pcbs/left_autorouted.kicad_pcb (KiCad board)
At the start: 2 copper layers, 123.1 x 93.2 mm, 29 parts

Commit message: Manually route the latest version:
Routing:
- net GND: track 113.0 -> 75.1 mm, vias 24 -> 23
Changed lines of the file:
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@@
 		(fp_arc
 			(start -19.286135 7.008046)
-			(mid -19.911512 4.959786)
+			(mid -19.911512 4.959785)
 			(end -20.32 2.8575)
 			(stroke
@@
 		(fp_line
 			(start 1.5 -3.7)
-			(end -0.8 -3.700003)
+			(end -0.8 -3.700002)
 			(stroke
 				(width 0.15)
@@
 			(start -2.5 -2.22)
 			(mid -1.956518 -3.312082)
-			(end -0.8 -3.700003)
+			(end -0.8 -3.700002)
 			(stroke
 				(width 0.15)
@@
 		)
 		(fp_line
-			(start -6.999997 -6)
+			(start -6.999998 -6)
 			(end -7 -7)
 			(stroke
@@
 		(fp_line
 			(start -7 7)
-			(end -6 6.999997)
+			(end -6 6.999998)
 			(stroke
 				(width 0.15)
@@
 		(fp_line
 			(start 7 -7)
-			(end 6 -6.999997)
+			(end 6 -6.999998)
 			(stroke
 				(width 0.15)
@@
 		)
 		(fp_line
-			(start 6.999997 6)
+			(start 6.999998 6)
 			(end 7 7)
 			(stroke
@@
 		(fp_line
 			(start 1.5 -3.7)
-			(end -0.8 -3.700003)
+			(end -0.8 -3.700002)
 			(stroke
 				(width 0.15)
@@
 			(start -2.5 -2.22)
 			(mid -1.956518 -3.312082)
-			(end -0.8 -3.700003)
+			(end -0.8 -3.700002)
 			(stroke
 				(width 0.15)
@@
 		)
 		(fp_line
-			(start -6.999997 -6)
+			(start -6.999998 -6)
 			(end -7 -7)
 			(stroke
@@
 		(fp_line
 			(start -7 7)
-			(end -6 6.999997)
+			(end -6 6.999998)
 			(stroke
 				(width 0.15)
@@
 		(fp_line
 			(start 7 -7)
-			(end 6 -6.999997)
+			(end 6 -6.999998)
 			(stroke
 				(width 0.15)
@@
 		)
 		(fp_line
-			(start 6.999997 6)
+			(start 6.999998 6)
 			(end 7 7)
 			(stroke
@@
 		(fp_arc
 			(start 2.52 -6.199998)
-			(mid 2.139877 -6.382303)
+			(mid 2.139878 -6.382304)
 			(end 2 -6.78)
 			(stroke
@@
 		(fp_arc
 			(start 2.52 -6.199998)
-			(mid 2.139877 -6.382303)
+			(mid 2.139878 -6.382304)
 			(end 2 -6.78)
 			(stroke
@@
 		(fp_arc
 			(start 2.52 -6.199998)
-			(mid 2.139877 -6.382303)
+			(mid 2.139878 -6.382304)
 			(end 2 -6.78)
 			(stroke
@@
 		(fp_line
 			(start 1.5 -3.7)
-			(end -0.8 -3.700003)
+			(end -0.8 -3.700002)
 			(stroke
 				(width 0.15)
@@
 			(start -2.5 -2.22)
 			(mid -1.956518 -3.312082)
-			(end -0.8 -3.700003)
+			(end -0.8 -3.700002)
 			(stroke
 				(width 0.15)
@@
 		)
 		(fp_line
-			(start -6.999997 -6)
+			(start -6.999998 -6)
 			(end -7 -7)
 			(stroke
@@
 		(fp_line
 			(start -7 7)
-			(end -6 6.999997)
+			(end -6 6.999998)
 			(stroke
 				(width 0.15)
@@
 		(fp_line
 			(start 7 -7)
-			(end 6 -6.999997)
+			(end 6 -6.999998)
 			(stroke
 				(width 0.15)
@@
 		)
 		(fp_line
-			(start 6.999997 6)
+			(start 6.999998 6)
 			(end 7 7)
 			(stroke
@@
 	)
 	(segment
-		(start 98.5235 111.8165)
-		(end 98.5235 114.7735)
-		(width 0.2)
-		(layer "F.Cu")
-		(net 2)
-	)
-	(segment
 		(start 196.4984 65.5643)
 		(end 196.498 65.5643)
@@
 	)
 	(segment
-		(start 190.074471 109.347201)
-		(end 189.102265 110.319407)
-		(width 0.2)
-		(layer "F.Cu")
-		(net 2)
-	)
-	(segment
 		(start 188.3234 63.0243)
 		(end 189.698 63.0243)
@@
 	)
 	(segment
-		(start 103.2696 114.619114)
-		(end 103.2696 114.2343)
-		(width 0.2)
-		(layer "F.Cu")
-		(net 2)
-	)
-	(segment
-		(start 98.91 115.16)
-		(end 102.728714 115.16)
-		(width 0.2)
-		(layer "F.Cu")
-		(net 2)
-	)
-	(segment
 		(start 188.323 63.0243)
 		(end 188.3234 63.0243)
@@
 	)
 	(segment
-		(start 102.728714 115.16)
-		(end 103.2696 114.619114)
-		(width 0.2)
-		(layer "F.Cu")
-		(net 2)
-	)
-	(segment
-		(start 189.102265 113.952265)
-		(end 194.34 119.19)
-		(width 0.2)
-		(layer "F.Cu")
-		(net 2)
-	)
-	(segment
-		(start 189.102265 110.319407)
-		(end 189.102265 113.952265)
-		(width 0.2)
-		(layer "F.Cu")
-		(net 2)
-	)
-	(segment
-		(start 101.6145 111.3343)
-		(end 99.0057 111.3343)
-		(width 0.2)
-		(layer "F.Cu")
-		(net 2)
-	)
-	(segment
-		(start 98.5235 114.7735)
-		(end 98.91 115.16)
-		(width 0.2)
-		(layer "F.Cu")
-		(net 2)
-	)
-	(segment
 		(start 197.873 68.1043)
 		(end 196.4984 68.1043)
@@
 		(net 2)
 	)
-	(segment
-		(start 99.0057 111.3343)
-		(end 98.5235 111.8165)
-		(width 0.2)
-		(layer "F.Cu")
-		(net 2)
-	)
-	(segment
-		(start 102.5145 112.2343)
-		(end 101.6145 111.3343)
-		(width 0.2)
-		(layer "F.Cu")
-		(net 2)
-	)
 	(via
 		(at 168.2206 39.7393)
@@
 	)
 	(via
-		(at 194.34 119.19)
-		(size 0.6)
-		(drill 0.3)
-		(layers "F.Cu" "B.Cu")
-		(net 2)
-	)
-	(via
 		(at 145.251 75.0064)
 		(size 0.6)
@@
 	)
 	(segment
-		(start 201.495516 120.056241)
-		(end 204.949513 116.602244)
-		(width 0.2)
-		(layer "B.Cu")
-		(net 2)
-	)
-	(segment
 		(start 187.5414 106.1173)
 		(end 187.1888 105.7647)
@@
 	)
 	(segment
-		(start 195.206241 120.056241)
-		(end 201.495516 120.056241)
-		(width 0.2)
-		(layer "B.Cu")
-		(net 2)
-	)
-	(segment
 		(start 124.8981 78.9705)
 		(end 124.8099 77.2871)
@@
 		(layer "B.Cu")
 		(net 2)
-	)
-	(segment
-		(start 194.34 119.19)
-		(end 195.206241 120.056241)
-		(width 0.2)
-		(layer "B.Cu")
-		(net 2)

Commit message: Update routes
Parts:
- removed TENTINGPUCK1: Tenting Puck, TentingPuck
Routing:
- net GND: track 75.1 -> 388.1 mm, vias 23 -> 24
- net P14: track 129.5 -> 146.9 mm, vias 2 -> 1
- net P16: track 99.6 -> 114.5 mm, vias 2 -> 1
- net P7: track 97.8 -> 83.4 mm, vias 2 -> 4
- net P10: track 115.3 -> 128.4 mm
- net P3: track 76.9 -> 86.1 mm
- net P18: track 128.2 -> 136.9 mm, vias 2 -> 3
- net P19: track 66.1 -> 58.6 mm
- net P1: track 47.1 -> 41.5 mm
- net P21: track 62.1 -> 67.3 mm
- net P0: track 41.9 -> 38.3 mm
- net P20: track 54.3 -> 57.8 mm
- net P15: track 115.9 -> 118.8 mm
- net P6: track 111.1 -> 113.3 mm
- net P9: track 130.9 -> 129.1 mm
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