File: pcbs/left_manually_routed.kicad_pcb (KiCad board)
At the start: 2 copper layers, 123.1 x 93.2 mm, 29 parts

Commit message: Update routes
Parts:
- removed TENTINGPUCK1: Tenting Puck, TentingPuck
Routing:
- net GND: track 113.0 -> 401.9 mm, vias 24 -> 25
- net P14: track 129.5 -> 146.9 mm, vias 2 -> 1
- net P16: track 99.6 -> 114.5 mm, vias 2 -> 1
- net P7: track 97.8 -> 83.4 mm, vias 2 -> 4
- net P10: track 115.3 -> 128.4 mm
- net P3: track 76.9 -> 86.1 mm
- net P18: track 128.2 -> 136.9 mm, vias 2 -> 3
- net P19: track 66.1 -> 58.6 mm
- net P1: track 47.1 -> 41.5 mm
- net P21: track 62.1 -> 67.3 mm
- net P0: track 41.9 -> 38.3 mm
- net P20: track 54.3 -> 57.8 mm
- net P15: track 115.9 -> 118.8 mm
- net P6: track 111.1 -> 113.3 mm
- net P9: track 130.9 -> 129.1 mm
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